File: IOB-I2C-MAX731x.sch (EAGLE design)
At the start: 9 parts, among them IC1 MAX7311, SW1 A0, SW2 A1, SW3 A2

Commit message: cleanup layout
Parts:
- BOARD: value I2C-EXPANDER -> CONNECTOR-I2C-EXPANDER; device SPCoast:I2C-EXPANDER -> SPCoast:CONNECTOR-I2C-EXPANDER
Changed lines of the file:
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@@
 <part name="P+5" library="supply1" deviceset="VCC" device=""/>
 <part name="P+10" library="supply1" deviceset="VCC" device=""/>
-<part name="BOARD" library="SPCoast" deviceset="I2C-EXPANDER" device=""/>
+<part name="BOARD" library="SPCoast" deviceset="CONNECTOR-I2C-EXPANDER" device=""/>
 <part name="C1" library="SPCoast" deviceset="CAP*" device="0603" value="0.1uF"/>
 <part name="P+1" library="supply1" deviceset="VCC" device=""/>

Commit message: normalized values
Parts:
- R17: device SPCoast:R0805-RES -> SPCoast:R0603-RES
- SW1: value A0 -> SPSTx4
- SW2: value A1 -> SPSTx4
- SW3: value A2 -> SPSTx4
- U$1: value DOC-OSHW-LOGO-L -> OSHW
Changed lines of the file:
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@@
 <layer number="20" name="Dimension" color="15" fill="1" visible="no" active="no"/>
 <layer number="21" name="tPlace" color="19" fill="1" visible="no" active="no"/>
-<layer number="22" name="bPlace" color="22" fill="1" visible="no" active="no"/>
+<layer number="22" name="bPlace" color="17" fill="1" visible="no" active="no"/>
 <layer number="23" name="tOrigins" color="30" fill="1" visible="no" active="no"/>
 <layer number="24" name="bOrigins" color="15" fill="1" visible="no" active="no"/>
@@
 <layer number="46" name="Milling" color="35" fill="1" visible="no" active="no"/>
 <layer number="47" name="Measures" color="21" fill="1" visible="no" active="no"/>
-<layer number="48" name="Document" color="57" fill="1" visible="no" active="no"/>
+<layer number="48" name="Document" color="47" fill="1" visible="no" active="no"/>
 <layer number="49" name="Reference" color="48" fill="1" visible="no" active="no"/>
 <layer number="50" name="dxf" color="7" fill="1" visible="no" active="no"/>
-<layer number="51" name="tDocu" color="49" fill="1" visible="no" active="no"/>
+<layer number="51" name="tDocu" color="24" fill="1" visible="no" active="no"/>
 <layer number="52" name="bDocu" color="7" fill="1" visible="no" active="no"/>
 <layer number="53" name="tGND_GNDA" color="7" fill="9" visible="no" active="no"/>
@@
 <parts>
 <part name="FRAME1" library="MCP" deviceset="FRAME-LETTER" device=""/>
-<part name="U$1" library="SPCoast" deviceset="DOC-OSHW-LOGO-" device="L" value="DOC-OSHW-LOGO-L"/>
+<part name="U$1" library="SPCoast" deviceset="DOC-OSHW-LOGO-" device="L" value="OSHW"/>
 <part name="V7" library="supply2" deviceset="GND" device=""/>
 <part name="P+6" library="supply1" deviceset="VCC" device=""/>
-<part name="R17" library="SPCoast" deviceset="R*" device="0805-RES" value="4k7"/>
+<part name="R17" library="SPCoast" deviceset="R*" device="0603-RES" value="4k7"/>
 <part name="LED16" library="SPCoast" deviceset="LED*" device="0603-LED" value="G"/>
 <part name="P+14" library="supply1" deviceset="VCC" device=""/>
@@
 <part name="V9" library="supply2" deviceset="GND" device=""/>
 <part name="IC1" library="SPCoast" deviceset="MAX73XX" device="/AUG" value="MAX7311"/>
-<part name="SW1" library="SPCoast" deviceset="SW_DIP-4" device="" value="A0"/>
-<part name="SW2" library="SPCoast" deviceset="SW_DIP-4" device="" value="A1"/>
-<part name="SW3" library="SPCoast" deviceset="SW_DIP-4" device="" value="A2"/>
+<part name="SW1" library="SPCoast" deviceset="SW_DIP-4" device="" value="SPSTx4"/>
+<part name="SW2" library="SPCoast" deviceset="SW_DIP-4" device="" value="SPSTx4"/>
+<part name="SW3" library="SPCoast" deviceset="SW_DIP-4" device="" value="SPSTx4"/>
 <part name="V5" library="supply2" deviceset="GND" device=""/>
 <part name="V6" library="supply2" deviceset="GND" device=""/>
